Commit message: Update trained checkpoint for KISTAR Hand

File: assets/kistar_right/model.urdf (robot description, URDF)
Before this commit: robot kistar_hand, 37 links, 36 joints
Joints:
- joint middle_joint_0: limit lower=-0.261799 upper=0.261799 effort=10.0 velocity=6.283 -> lower=-0.081799 upper=0.081799 effort=10.0 velocity=6.283
